File: sch/double-action-keyboard/double-action-keyboard.kicad_pcb (KiCad board)
At the start: 2 copper layers, 132 x 85 mm, 151 parts, among them J1 Conn_01x02, J2 Conn_01x04, J3 Conn_01x04, U1 Pico, U2 AQM1602XA-RN-GBW, U3 AQM1602Y-NLW-FBW

Commit message: LCD(小)とOLEDを同時に実装できるように位置を調整しました。 スイッチのランドを0.5mm大きくしました。
Parts:
- moved R4 20.3 mm to (91.0, 49.0)
- moved C4 17.1 mm to (106.0, 49.0)
- moved C5 17.1 mm to (98.0, 49.0)
- moved C6 17.1 mm to (102.0, 49.0)
- moved U3 15.8 mm to (104.0, 53.0)
- moved R6 12.9 mm to (113.0, 49.0), turned to 0 degrees
- moved R5 12.6 mm to (117.0, 49.0)
- moved J3 11.7 mm to (97.5, 27.0)
- moved J2 10.6 mm to (72.0, 27.0)
- moved C8 10.4 mm to (66.0, 30.0)
- moved C7 9.51 mm to (66.0, 33.0)
- moved C10 8.00 mm to (98.0, 31.0), turned to 0 degrees
- moved C9 8.00 mm to (98.0, 33.0), turned to 0 degrees
- moved C3 1.00 mm to (93.1, 34.0)
Routing:
- net /LCD_I2C_SCL: track 126.2 -> 157.5 mm
- net +3.3V: track 176.9 -> 206.4 mm, vias 9 -> 8
- net /LCD_I2C_SDA: track 122.1 -> 138.6 mm
- net Net-(U2-CAP1N): track 3.24 -> 5.11 mm
- net Net-(U2-CAP1P): track 2.75 -> 3.91 mm
- net Net-(U3-CAP1N): track 4.39 -> 4.92 mm
- net Net-(U3-CAP1P): track 4.05 -> 4.58 mm
- net (no net): vias 109 -> 78
